File: Daisy_MultiEffect_Pedal_KiCad_Starter/Daisy_MultiEffect_Pedal.kicad_pcb (KiCad board)
At the start: 2 copper layers, 150 x 90 mm, 24 parts, among them J1 INPUT_TS_JACK, J2 OUTPUT_TS_JACK, SW1 MOMENTARY_MODE_SWITCH, U1 MCP6002-I/P, U2 Daisy Seed socket / 2x20

Commit message: made fixes to schematic and pcb design, added readme
Parts:
- RV5: value B10K -> B10K volume
- moved RV5 57.8 mm to (120.0, 68.0)
Connections:
- C7 pad 2: OUT_JACK_TIP -> OUT_LEVEL_IN
- RV5 pad 2: POT5_A4_D19 -> OUT_JACK_TIP
- RV5 pad 3: +3V3A -> OUT_LEVEL_IN
- U2 pad 26: POT5_A4_D19 -> (no net)
Routing:
- net GND: track 0.00 -> 479.8 mm
- net D9_SWITCH: track 0.00 -> 196.7 mm
- net +3V3A: track 0.00 -> 175.4 mm
- net POT1_A0_D15: track 0.00 -> 136.3 mm
- net POT2_A1_D16: track 0.00 -> 116.9 mm
- net VREF_1V65: track 0.00 -> 111.0 mm
- net POT3_A2_D17: track 0.00 -> 97.4 mm
- net POT4_A3_D18: track 0.00 -> 77.9 mm
- net OUT_JACK_TIP: track 0.00 -> 72.7 mm
- net OUT_BUF_INPUT: track 0.00 -> 59.8 mm, vias 0 -> 1
- net INPUT_NODE: track 0.00 -> 43.0 mm
- net AUDIO_IN_L: track 0.00 -> 40.3 mm
- net OUT_BUF_OUT: track 0.00 -> 39.2 mm
- net AUDIO_OUT_L: track 0.00 -> 27.0 mm
- net OUT_LEVEL_IN: track 0.00 -> 22.7 mm
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Other:
- board text added: "RV5 = wired output volume. RV1-RV4 are optional ADC headers not used by current firmware."

Commit message: fixed PCB and schematic files, finalized PCB design for ordering
Parts:
- moved SW1 86.3 mm to (106.0, 34.0)
- moved RV5 23.4 mm to (105.0, 86.0)
- moved J2 13.0 mm to (140.0, 86.0)
Routing:
- net D9_SWITCH: track 196.7 -> 33.4 mm
- net OUT_JACK_TIP: track 72.7 -> 48.0 mm
- net OUT_BUF_INPUT: track 59.8 -> 83.8 mm, vias 1 -> 0
- net +3V3A: track 175.4 -> 164.1 mm
- net GND: track 479.8 -> 488.3 mm
- net OUT_LEVEL_IN: track 22.7 -> 15.7 mm
- net IN_JACK_TIP: track 17.7 -> 23.7 mm
- net VREF_1V65: track 111.0 -> 116.0 mm
- net POT4_A3_D18: track 77.9 -> 75.9 mm
Other:
- board text added: "Daisy Seed Multi-Effect Pedal STARTER PCB"
- board text removed: "Daisy Seed Multi-Effect Pedal STARTER PCB - inspect before fabrication"
