File: Daisy_MultiEffect_Pedal_KiCad_Starter/Daisy_MultiEffect_Pedal.kicad_sch (KiCad schematic)
At the start: 24 parts, among them J1 Input TS jack: tip/sleeve, J2 Output TS jack: tip/sleeve, SW1 Momentary mode switch, U1 MCP6002 dual op-amp, U2 Daisy Seed minimal pinout

Commit message: made fixes to schematic and pcb design, added readme
Connections:
- net +3V3A: now also C3.1, R1.1, RV1.1 (GND), RV2.1 (GND), RV3.1 (GND), RV4.1 (GND), U1.4 (VSS)
- net AUDIO_IN_L: now also C5.2
- net AUDIO_OUT_L: now also C6.1
- net AUDIO_OUT_R_UNUSED: now also U2.19 (AUDIO_OUT_R)
- net BUF_IN_OUT: now also R4.1
- net BUF_TO_DAISY_C: now also C5.1, R4.2
- net D9_SWITCH: now also SW1.1
- net GND: now also C1.2, C2.2, C3.2, J1.2, J2.2, R2.2, R7.2, RV1.3 (3V3), RV2.3 (3V3), RV3.3 (3V3), RV4.3 (3V3), RV5.3 (3V3), SW1.2, U1.8 (VDD)
- net INPUT_NODE: now also C4.2, R3.1, U1.3 (IN+_A)
- net IN_JACK_TIP: now also C4.1, J1.1
- net OUT_BUF_INPUT: now also C6.2, R5.1, U1.5 (IN+_B)
- net OUT_BUF_OUT: now also R6.1
- net OUT_CAP_IN: now also C7.1, R6.2
- net OUT_JACK_TIP: now also J2.1, R7.1, RV5.2 (WIPER)
- net POT1_A0_D15: now also RV1.2 (WIPER)
- net POT2_A1_D16: now also RV2.2 (WIPER)
- net POT3_A2_D17: now also RV3.2 (WIPER)
- net POT4_A3_D18: now also RV4.2 (WIPER)
- net VREF_1V65: now also C1.1, C2.1, R1.2, R2.1, R3.2, R5.2
- net OUT_LEVEL_IN: now reaches C7.2
- net OUT_LEVEL_IN: now also RV5.1 (GND)
Other:
- note added: "RV5 is output volume: 1=GND, 2=wiper to output jack, 3=post-output-cap. RV1-RV4 are optional future ADC controls."
- note removed: "Pot pins: 1=GND, 2=wiper to ADC, 3=+3V3A. Your current C++ does not read these yet."

Commit message: fixed PCB and schematic files, finalized PCB design for ordering
Connections:
- net +3V3A: now also U1.8 (VDD), U2.21 (+3V3A); no longer U1.4 (VSS)
- net AUDIO_IN_L: now also U2.16 (AUDIO_IN_L)
- net AUDIO_OUT_L: now also U2.18 (AUDIO_OUT_L)
- net BUF_IN_OUT: now also U1.1 (OUT_A), U1.2 (IN-_A)
- net D9_SWITCH: now also U2.10 (D9)
- net GND: now also U1.4 (VSS), U2.20 (AGND), U2.40 (DGND); no longer U1.8 (VDD)
- net OUT_BUF_OUT: now also U1.6 (IN-_B), U1.7 (OUT_B)
- net POT1_A0_D15: now also U2.22 (A0_D15)
- net POT2_A1_D16: now also U2.23 (A1_D16)
- net POT3_A2_D17: now also U2.24 (A2_D17)
- net POT4_A3_D18: now also U2.25 (A3_D18)
Other:
- note removed: "This file is a reviewable KiCad starter, not a production-ready design. Run ERC/DRC and verify footprints/pinouts."
